File: KiCad/60_Keyboard.kicad_pcb (KiCad board)
At the start: 2 copper layers, 285.7 x 95.2 mm, 153 parts, among them SW1 SW_Push, U1 ATmega32U4-A, Y1 16MHz

Commit message: Made the keyboard Back
Other:
- board text added: "60"
- board text added: "Circuits Unleased"
- board text added: "Designed By Lucien Lee"

Commit message: changes to gerber files and uploads of stl files that will be used
Other:
- board text added: "*"
Changed lines of the file:
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@@
 		(layer "Edge.Cuts")
+	)
+	(gr_text "*\n"
+		(at 108.7369 100.0062 0)
+		(layer "B.SilkS")
+		(effects
+			(font
+				(size 1 1)
+				(thickness 0.1)
+			)
+			(justify left bottom mirror)
+		)
 	)
 	(gr_text "Designed By Lucien Lee\n"
